Commit message: Traffic police monitor speed

File: src/delivery_robot_description/models/delivery_robot/delivery_robot.urdf.xacro (robot description, xacro)
@@ -15,5 +15,5 @@
     <xacro:imu_xacro xyz="0.0 0.0 0.18"/>
     <xacro:laser_xacro xyz="0.0 0.0 0.28"/>
-    <xacro:camera_xacro xyz="0.36 0.0 0.15"/>
+    <xacro:stereo_camera_xacro xyz="0.36 0.0 0.15" baseline="0.12"/>
     <xacro:wheel_xacro wheel_name="left_wheel" xyz="0 0.36 -0.12" />
     <xacro:wheel_xacro wheel_name="right_wheel" xyz="0 -0.36 -0.12" />

File: src/delivery_robot_description/models/delivery_robot/plugin/gz_sensor_plugin.xacro (robot description, xacro)
@@ -100,12 +100,43 @@
             </sensor>
         </gazebo>
-        <gazebo reference="camera_link">
-            <sensor name="camera_sensor" type="camera">
-                <topic>/delivery_robot/camera/image_raw</topic>
-                <gz_frame_id>camera_link</gz_frame_id>
+        <gazebo reference="left_camera_link">
+            <sensor name="left_camera_sensor" type="camera">
+                <topic>/delivery_robot/stereo/left/image_raw</topic>
+                <gz_frame_id>left_camera_optical_link</gz_frame_id>
                 <always_on>true</always_on>
+                <visualize>true</visualize>
                 <update_rate>10</update_rate>
-                <camera name="camera">
-                    <camera_info_topic>/delivery_robot/camera/camera_info</camera_info_topic>
+                <camera name="left_camera">
+                    <camera_info_topic>/delivery_robot/stereo/left/camera_info</camera_info_topic>
+                    <horizontal_fov>1.5009831567</horizontal_fov>
+                    <image>
+                        <width>800</width>
+                        <height>600</height>
+                        <format>R8G8B8</format>
+                    </image>
+                    <clip>
+                        <near>0.12</near>
+                        <far>8.0</far>
+                    </clip>
+                    <distortion>
+                        <k1>0.0</k1>
+                        <k2>0.0</k2>
+                        <k3>0.0</k3>
+                        <p1>0.0</p1>
+                        <p2>0.0</p2>
+                        <center>0.5 0.5</center>
+                    </distortion>
+                </camera>
+            </sensor>
+        </gazebo>
+        <gazebo reference="right_camera_link">
+            <sensor name="right_camera_sensor" type="camera">
+                <topic>/delivery_robot/stereo/right/image_raw</topic>
+                <gz_frame_id>right_camera_optical_link</gz_frame_id>
+                <always_on>true</always_on>
+                <visualize>true</visualize>
+                <update_rate>10</update_rate>
+                <camera name="right_camera">
+                    <camera_info_topic>/delivery_robot/stereo/right/camera_info</camera_info_topic>
                     <horizontal_fov>1.5009831567</horizontal_fov>
                     <image>

File: src/delivery_robot_description/models/delivery_robot/sensor/camera.urdf.xacro (robot description, xacro)
@@ -2,13 +2,13 @@
 <robot xmlns:xacro="http://www.ros.org/wiki/xacro">
     <xacro:include filename="$(find delivery_robot_description)/models/delivery_robot/common_inertia.xacro" />
-    <xacro:macro name="camera_xacro" params="xyz">
-        <link name="camera_link">
+    <xacro:macro name="stereo_camera_xacro" params="xyz baseline">
+        <link name="stereo_camera_link">
             <visual>
                 <origin xyz="0.0 0.0 0.0" rpy="0.0 0.0 0.0"/>
                 <geometry>
-                    <box size="0.12 0.18 0.12"/>
+                    <box size="0.12 ${baseline + 0.10} 0.10"/>
                 </geometry>
                 <material name="black">
-                    <color rgba="0.0 0.0 0.0 0.5"/>
+                    <color rgba="0.0 0.0 0.0 0.8"/>
                 </material>
             </visual>
@@ -16,22 +16,55 @@
                 <origin xyz="0.0 0.0 0.0" rpy="0.0 0.0 0.0"/>
                 <geometry>
-                    <box size="0.12 0.18 0.12"/>
+                    <box size="0.12 ${baseline + 0.10} 0.10"/>
                 </geometry>
-                <material name="black">
-                    <color rgba="0.0 0.0 0.0 0.5"/>
+            </collision>
+            <xacro:box_inertia m="0.2" w="0.12" h="${baseline + 0.10}" d="0.10" />
+        </link>
+        <link name="left_camera_link">
+            <visual>
+                <geometry>
+                    <cylinder radius="0.035" length="0.04"/>
+                </geometry>
+                <origin xyz="0.04 0 0" rpy="0 ${pi / 2.0} 0"/>
+                <material name="camera_lens">
+                    <color rgba="0.05 0.10 0.20 1.0"/>
                 </material>
-            </collision>
-            <xacro:box_inertia m="0.2" w="0.12" h="0.18" d="0.12" />
+            </visual>
         </link>
-        <link name="camera_optical_link" />
-        <joint name="camera_joint" type="fixed">
+        <link name="right_camera_link">
+            <visual>
+                <geometry>
+                    <cylinder radius="0.035" length="0.04"/>
+                </geometry>
+                <origin xyz="0.04 0 0" rpy="0 ${pi / 2.0} 0"/>
+                <material name="camera_lens"/>
+            </visual>
+        </link>
+        <link name="left_camera_optical_link"/>
+        <link name="right_camera_optical_link"/>
+        <joint name="stereo_camera_joint" type="fixed">
             <parent link="base_link"/>
-            <child link="camera_link"/>
+            <child link="stereo_camera_link"/>
             <origin xyz="${xyz}" rpy="0.0 0.0 0.0"/>
         </joint>
-        <joint name="camera_optical_joint" type="fixed">
-            <parent link="camera_link"/>
-            <child link="camera_optical_link"/>
-            <origin xyz="0 0 0" rpy="0.0 0.0 0.0"/>
+        <joint name="left_camera_joint" type="fixed">
+            <parent link="stereo_camera_link"/>
+            <child link="left_camera_link"/>
+            <origin xyz="0 ${baseline / 2.0} 0" rpy="0.0 0.0 0.0"/>
+        </joint>
+        <joint name="right_camera_joint" type="fixed">
+            <parent link="stereo_camera_link"/>
+            <child link="right_camera_link"/>
+            <origin xyz="0 ${-baseline / 2.0} 0" rpy="0.0 0.0 0.0"/>
+        </joint>
+        <joint name="left_camera_optical_joint" type="fixed">
+            <parent link="left_camera_link"/>
+            <child link="left_camera_optical_link"/>
+            <origin xyz="0 0 0" rpy="${-pi / 2.0} 0 ${-pi / 2.0}"/>
+        </joint>
+        <joint name="right_camera_optical_joint" type="fixed">
+            <parent link="right_camera_link"/>
+            <child link="right_camera_optical_link"/>
+            <origin xyz="0 0 0" rpy="${-pi / 2.0} 0 ${-pi / 2.0}"/>
         </joint>
     </xacro:macro>

Commit message: Traffic police monitor speed

File: src/delivery_robot_description/models/delivery_robot/delivery_robot.urdf.xacro (robot description, xacro)
@@ -15,5 +15,5 @@
     <xacro:imu_xacro xyz="0.0 0.0 0.18"/>
     <xacro:laser_xacro xyz="0.0 0.0 0.28"/>
-    <xacro:stereo_camera_xacro xyz="0.36 0.0 0.15" baseline="0.12"/>
+    <xacro:rgbd_camera_xacro xyz="0.36 0.0 0.15"/>
     <xacro:wheel_xacro wheel_name="left_wheel" xyz="0 0.36 -0.12" />
     <xacro:wheel_xacro wheel_name="right_wheel" xyz="0 -0.36 -0.12" />

File: src/delivery_robot_description/models/delivery_robot/plugin/gz_sensor_plugin.xacro (robot description, xacro)
@@ -100,13 +100,17 @@
             </sensor>
         </gazebo>
-        <gazebo reference="left_camera_link">
-            <sensor name="left_camera_sensor" type="camera">
-                <topic>/delivery_robot/stereo/left/image_raw</topic>
-                <gz_frame_id>left_camera_optical_link</gz_frame_id>
+        <gazebo reference="rgbd_camera_link">
+            <sensor name="rgbd_camera_sensor" type="rgbd_camera">
+                <!--
+                  RGB-D sensors append /image and /depth_image to this base
+                  topic. Both streams share the same optical frame and clock.
+                -->
+                <topic>/delivery_robot/rgbd</topic>
+                <gz_frame_id>rgbd_camera_optical_link</gz_frame_id>
                 <always_on>true</always_on>
                 <visualize>true</visualize>
                 <update_rate>10</update_rate>
-                <camera name="left_camera">
-                    <camera_info_topic>/delivery_robot/stereo/left/camera_info</camera_info_topic>
+                <camera name="rgbd_camera">
+                    <camera_info_topic>/delivery_robot/rgbd/camera_info</camera_info_topic>
                     <horizontal_fov>1.5009831567</horizontal_fov>
                     <image>
@@ -119,34 +123,10 @@
                         <far>8.0</far>
                     </clip>
-                    <distortion>
-                        <k1>0.0</k1>
-                        <k2>0.0</k2>
-                        <k3>0.0</k3>
-                        <p1>0.0</p1>
-                        <p2>0.0</p2>
-                        <center>0.5 0.5</center>
-                    </distortion>
-                </camera>
-            </sensor>
-        </gazebo>
-        <gazebo reference="right_camera_link">
-            <sensor name="right_camera_sensor" type="camera">
-                <topic>/delivery_robot/stereo/right/image_raw</topic>
-                <gz_frame_id>right_camera_optical_link</gz_frame_id>
-                <always_on>true</always_on>
-                <visualize>true</visualize>
-                <update_rate>10</update_rate>
-                <camera name="right_camera">
-                    <camera_info_topic>/delivery_robot/stereo/right/camera_info</camera_info_topic>
-                    <horizontal_fov>1.5009831567</horizontal_fov>
-                    <image>
-                        <width>800</width>
-                        <height>600</height>
-                        <format>R8G8B8</format>
-                    </image>
-                    <clip>
-                        <near>0.12</near>
-                        <far>8.0</far>
-                    </clip>
+                    <depth_camera>
+                        <clip>
+                            <near>0.12</near>
+                            <far>8.0</far>
+                        </clip>
+                    </depth_camera>
                     <distortion>
                         <k1>0.0</k1>

File: src/delivery_robot_description/models/delivery_robot/sensor/camera.urdf.xacro (robot description, xacro)
@@ -2,10 +2,10 @@
 <robot xmlns:xacro="http://www.ros.org/wiki/xacro">
     <xacro:include filename="$(find delivery_robot_description)/models/delivery_robot/common_inertia.xacro" />
-    <xacro:macro name="stereo_camera_xacro" params="xyz baseline">
-        <link name="stereo_camera_link">
+    <xacro:macro name="rgbd_camera_xacro" params="xyz">
+        <link name="rgbd_camera_link">
             <visual>
                 <origin xyz="0.0 0.0 0.0" rpy="0.0 0.0 0.0"/>
                 <geometry>
-                    <box size="0.12 ${baseline + 0.10} 0.10"/>
+                    <box size="0.12 0.20 0.10"/>
                 </geometry>
                 <material name="black">
@@ -14,56 +14,19 @@
             </visual>
             <collision>
-                <origin xyz="0.0 0.0 0.0" rpy="0.0 0.0 0.0"/>
                 <geometry>
-                    <box size="0.12 ${baseline + 0.10} 0.10"/>
+                    <box size="0.12 0.20 0.10"/>
                 </geometry>
             </collision>
-            <xacro:box_inertia m="0.2" w="0.12" h="${baseline + 0.10}" d="0.10" />
+            <xacro:box_inertia m="0.2" w="0.12" h="0.20" d="0.10"/>
         </link>
-        <link name="left_camera_link">
-            <visual>
-                <geometry>
-                    <cylinder radius="0.035" length="0.04"/>
-                </geometry>
-                <origin xyz="0.04 0 0" rpy="0 ${pi / 2.0} 0"/>
-                <material name="camera_lens">
-                    <color rgba="0.05 0.10 0.20 1.0"/>
-                </material>
-            </visual>
-        </link>
-        <link name="right_camera_link">
-            <visual>
-                <geometry>
-                    <cylinder radius="0.035" length="0.04"/>
-                </geometry>
-                <origin xyz="0.04 0 0" rpy="0 ${pi / 2.0} 0"/>
-                <material name="camera_lens"/>
-            </visual>
-        </link>
-        <link name="left_camera_optical_link"/>
-        <link name="right_camera_optical_link"/>
-        <joint name="stereo_camera_joint" type="fixed">
+        <link name="rgbd_camera_optical_link"/>
+        <joint name="rgbd_camera_joint" type="fixed">
             <parent link="base_link"/>
-            <child link="stereo_camera_link"/>
+            <child link="rgbd_camera_link"/>
             <origin xyz="${xyz}" rpy="0.0 0.0 0.0"/>
         </joint>
-        <joint name="left_camera_joint" type="fixed">
-            <parent link="stereo_camera_link"/>
-            <child link="left_camera_link"/>
-            <origin xyz="0 ${baseline / 2.0} 0" rpy="0.0 0.0 0.0"/>
-        </joint>
-        <joint name="right_camera_joint" type="fixed">
-            <parent link="stereo_camera_link"/>
-            <child link="right_camera_link"/>
-            <origin xyz="0 ${-baseline / 2.0} 0" rpy="0.0 0.0 0.0"/>
-        </joint>
-        <joint name="left_camera_optical_joint" type="fixed">
-            <parent link="left_camera_link"/>
-            <child link="left_camera_optical_link"/>
-            <origin xyz="0 0 0" rpy="${-pi / 2.0} 0 ${-pi / 2.0}"/>
-        </joint>
-        <joint name="right_camera_optical_joint" type="fixed">
-            <parent link="right_camera_link"/>
-            <child link="right_camera_optical_link"/>
+        <joint name="rgbd_camera_optical_joint" type="fixed">
+            <parent link="rgbd_camera_link"/>
+            <child link="rgbd_camera_optical_link"/>
             <origin xyz="0 0 0" rpy="${-pi / 2.0} 0 ${-pi / 2.0}"/>
         </joint>

Commit message: [FEAT]: Traffic police monitor speed (#5)

File: src/delivery_robot_description/models/delivery_robot/delivery_robot.urdf.xacro (robot description, xacro)
@@ -15,5 +15,5 @@
     <xacro:imu_xacro xyz="0.0 0.0 0.18"/>
     <xacro:laser_xacro xyz="0.0 0.0 0.28"/>
-    <xacro:camera_xacro xyz="0.36 0.0 0.15"/>
+    <xacro:rgbd_camera_xacro xyz="0.36 0.0 0.15"/>
     <xacro:wheel_xacro wheel_name="left_wheel" xyz="0 0.36 -0.12" />
     <xacro:wheel_xacro wheel_name="right_wheel" xyz="0 -0.36 -0.12" />

File: src/delivery_robot_description/models/delivery_robot/plugin/gz_sensor_plugin.xacro (robot description, xacro)
@@ -100,12 +100,17 @@
             </sensor>
         </gazebo>
-        <gazebo reference="camera_link">
-            <sensor name="camera_sensor" type="camera">
-                <topic>/delivery_robot/camera/image_raw</topic>
-                <gz_frame_id>camera_link</gz_frame_id>
+        <gazebo reference="rgbd_camera_link">
+            <sensor name="rgbd_camera_sensor" type="rgbd_camera">
+                <!--
+                  RGB-D sensors append /image and /depth_image to this base
+                  topic. Both streams share the same optical frame and clock.
+                -->
+                <topic>/delivery_robot/rgbd</topic>
+                <gz_frame_id>rgbd_camera_optical_link</gz_frame_id>
                 <always_on>true</always_on>
+                <visualize>true</visualize>
                 <update_rate>10</update_rate>
-                <camera name="camera">
-                    <camera_info_topic>/delivery_robot/camera/camera_info</camera_info_topic>
+                <camera name="rgbd_camera">
+                    <camera_info_topic>/delivery_robot/rgbd/camera_info</camera_info_topic>
                     <horizontal_fov>1.5009831567</horizontal_fov>
                     <image>
@@ -118,4 +123,10 @@
                         <far>8.0</far>
                     </clip>
+                    <depth_camera>
+                        <clip>
+                            <near>0.12</near>
+                            <far>8.0</far>
+                        </clip>
+                    </depth_camera>
                     <distortion>
                         <k1>0.0</k1>

File: src/delivery_robot_description/models/delivery_robot/sensor/camera.urdf.xacro (robot description, xacro)
@@ -2,36 +2,32 @@
 <robot xmlns:xacro="http://www.ros.org/wiki/xacro">
     <xacro:include filename="$(find delivery_robot_description)/models/delivery_robot/common_inertia.xacro" />
-    <xacro:macro name="camera_xacro" params="xyz">
-        <link name="camera_link">
+    <xacro:macro name="rgbd_camera_xacro" params="xyz">
+        <link name="rgbd_camera_link">
             <visual>
                 <origin xyz="0.0 0.0 0.0" rpy="0.0 0.0 0.0"/>
                 <geometry>
-                    <box size="0.12 0.18 0.12"/>
+                    <box size="0.12 0.20 0.10"/>
                 </geometry>
                 <material name="black">
-                    <color rgba="0.0 0.0 0.0 0.5"/>
+                    <color rgba="0.0 0.0 0.0 0.8"/>
                 </material>
             </visual>
             <collision>
-                <origin xyz="0.0 0.0 0.0" rpy="0.0 0.0 0.0"/>
                 <geometry>
-                    <box size="0.12 0.18 0.12"/>
+                    <box size="0.12 0.20 0.10"/>
                 </geometry>
-                <material name="black">
-                    <color rgba="0.0 0.0 0.0 0.5"/>
-                </material>
             </collision>
-            <xacro:box_inertia m="0.2" w="0.12" h="0.18" d="0.12" />
+            <xacro:box_inertia m="0.2" w="0.12" h="0.20" d="0.10"/>
         </link>
-        <link name="camera_optical_link" />
-        <joint name="camera_joint" type="fixed">
+        <link name="rgbd_camera_optical_link"/>
+        <joint name="rgbd_camera_joint" type="fixed">
             <parent link="base_link"/>
-            <child link="camera_link"/>
+            <child link="rgbd_camera_link"/>
             <origin xyz="${xyz}" rpy="0.0 0.0 0.0"/>
         </joint>
-        <joint name="camera_optical_joint" type="fixed">
-            <parent link="camera_link"/>
-            <child link="camera_optical_link"/>
-            <origin xyz="0 0 0" rpy="0.0 0.0 0.0"/>
+        <joint name="rgbd_camera_optical_joint" type="fixed">
+            <parent link="rgbd_camera_link"/>
+            <child link="rgbd_camera_optical_link"/>
+            <origin xyz="0 0 0" rpy="${-pi / 2.0} 0 ${-pi / 2.0}"/>
         </joint>
     </xacro:macro>
